File: afterdark/bizcard-afterdark-1206-ledcoincell-no-resistor.kicad_pcb (KiCad board)
At the start: 2 copper layers, 35.9 x 20.8 mm, 4 parts

Commit message: add 1206 LED variation
Parts:
- REF**: value LED_0805_2012Metric_Pad1.15x1.40mm_HandSolder -> LED_1206_3216Metric_Pad1.42x1.75mm_HandSolder; footprint LED_SMD:LED_0805_2012Metric_Pad1.15x1.40mm_HandSolder -> LED_SMD:LED_1206_3216Metric_Pad1.42x1.75mm_HandSolder
Changed lines of the file:
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@@
     (uvia_drill 0.1)
   )
-  (module LED_SMD:LED_0805_2012Metric_Pad1.15x1.40mm_HandSolder (layer B.Cu)
+  (module LED_SMD:LED_1206_3216Metric_Pad1.42x1.75mm_HandSolder (layer B.Cu)
     (at 144.6276 70.358)
-    (descr "LED SMD 0805 (2012 Metric), square (rectangular) end terminal, IPC_7351 nominal, (Body size source: https://docs.google.com/spreadsheets/d/1BsfQQcO9C6DZCsRaXUlFlo91Tg2WpOkGARC1WS5S8t0/edit?usp=sharing), generated with kicad-footprint-generator")
+    (descr "LED SMD 1206 (3216 Metric), square (rectangular) end terminal, IPC_7351 nominal, (Body size source: http://www.tortai-tech.com/upload/download/2011102023233369053.pdf), generated with kicad-footprint-generator")
     (tags "LED handsolder")
     (attr smd)
@@
       (effects (font (size 1 1) (thickness 0.15)) (justify mirror))
     )
-    (fp_text value LED_0805_2012Metric_Pad1.15x1.40mm_HandSolder (at 0 -1.65 180) (layer B.Fab) hide
+    (fp_text value LED_1206_3216Metric_Pad1.42x1.75mm_HandSolder (at 0 -1.65 180) (layer B.Fab) hide
       (effects (font (size 1 1) (thickness 0.15)) (justify mirror))
     )
@@
       (effects (font (size 0.5 0.5) (thickness 0.08)) (justify mirror))
     )
-    (fp_line (start 1.85 -0.95) (end -1.85 -0.95) (layer B.CrtYd) (width 0.05))
-    (fp_line (start 1.85 0.95) (end 1.85 -0.95) (layer B.CrtYd) (width 0.05))
-    (fp_line (start -1.85 0.95) (end 1.85 0.95) (layer B.CrtYd) (width 0.05))
-    (fp_line (start -1.85 -0.95) (end -1.85 0.95) (layer B.CrtYd) (width 0.05))
-    (fp_line (start 1 -0.6) (end 1 0.6) (layer B.Fab) (width 0.1))
-    (fp_line (start -1 -0.6) (end 1 -0.6) (layer B.Fab) (width 0.1))
-    (fp_line (start -1 0.3) (end -1 -0.6) (layer B.Fab) (width 0.1))
-    (fp_line (start -0.7 0.6) (end -1 0.3) (layer B.Fab) (width 0.1))
-    (fp_line (start 1 0.6) (end -0.7 0.6) (layer B.Fab) (width 0.1))
-    (fp_text user + (at -2.1844 -0.7112) (layer B.Cu)
+    (fp_line (start 2.45 -1.12) (end -2.45 -1.12) (layer B.CrtYd) (width 0.05))
+    (fp_line (start 2.45 1.12) (end 2.45 -1.12) (layer B.CrtYd) (width 0.05))
+    (fp_line (start -2.45 1.12) (end 2.45 1.12) (layer B.CrtYd) (width 0.05))
+    (fp_line (start -2.45 -1.12) (end -2.45 1.12) (layer B.CrtYd) (width 0.05))
+    (fp_line (start -2.46 -1.135) (end 1.6 -1.135) (layer B.SilkS) (width 0.12))
+    (fp_line (start -2.46 1.135) (end -2.46 -1.135) (layer B.SilkS) (width 0.12))
+    (fp_line (start 1.6 1.135) (end -2.46 1.135) (layer B.SilkS) (width 0.12))
+    (fp_line (start 1.6 -0.8) (end 1.6 0.8) (layer B.Fab) (width 0.1))
+    (fp_line (start -1.6 -0.8) (end 1.6 -0.8) (layer B.Fab) (width 0.1))
+    (fp_line (start -1.6 0.4) (end -1.6 -0.8) (layer B.Fab) (width 0.1))
+    (fp_line (start -1.2 0.8) (end -1.6 0.4) (layer B.Fab) (width 0.1))
+    (fp_line (start 1.6 0.8) (end -1.2 0.8) (layer B.Fab) (width 0.1))
+    (fp_text user + (at -3.048 -0.8382) (layer B.Cu)
       (effects (font (size 0.5 0.5) (thickness 0.1)) (justify mirror))
     )
-    (pad 2 smd roundrect (at 1.025 0) (size 1.15 1.4) (layers B.Cu B.Paste B.Mask) (roundrect_rratio 0.217391))
-    (pad 1 smd roundrect (at -1.025 0) (size 1.15 1.4) (layers B.Cu B.Paste B.Mask) (roundrect_rratio 0.217391))
-    (model ${KISYS3DMOD}/LED_SMD.3dshapes/LED_0805_2012Metric.wrl
+    (pad 2 smd roundrect (at 1.4875 0) (size 1.425 1.75) (layers B.Cu B.Paste B.Mask) (roundrect_rratio 0.175439))
+    (pad 1 smd roundrect (at -1.4875 0) (size 1.425 1.75) (layers B.Cu B.Paste B.Mask) (roundrect_rratio 0.175439))
+    (model ${KISYS3DMOD}/LED_SMD.3dshapes/LED_1206_3216Metric.wrl
       (at (xyz 0 0 0))
       (scale (xyz 1 1 1))
