File: flex-bizcard/flex-strip-tester-v2.kicad_pcb (KiCad board)
At the start: 2 copper layers, 67.2 x 11.1 mm, 6 parts, among them J1 Conn_01x01_Female, J2 Conn_01x01_Female

Commit message: update flex tester
Routing:
- net GND: vias 0 -> 1
- net +3V3: vias 0 -> 1
- added copper zone on F.Cu, net +3V3
- removed copper zone on F.Cu, net GND
